Commit message: ✨ feat: urdf修正

File: config/robot.urdf (robot description, URDF)
Before this commit: robot bupt_dog, 17 links, 16 joints
Links:
- link FL_FOOT: mass 0.0 -> 0.06
- link FR_FOOT: mass 0.0 -> 0.06
- link HL_FOOT: mass 0.0 -> 0.06
- link HR_FOOT: mass 0.0 -> 0.06
- link body: mass 7.863 -> 7.1; geometry collision box size=0.322 0.22 0.115; visual box size=0.322 0.22 0.115
Joints:
- joint FL_FOOT_joint: origin xyz=0.0 0.0 -0.228 rpy=0.0 0.0 0.0 -> xyz=0.0 0.0 -0.24944 rpy=0.0 0.0 0.0
- joint FL_X_joint: origin xyz=0.240292 0.056 0 rpy=0 0 0 -> xyz=0.216 0.048 0 rpy=0 0 0
- joint FR_FOOT_joint: origin xyz=0.0 0.0 -0.228 rpy=0.0 0.0 0.0 -> xyz=0.0 0.0 -0.24944 rpy=0.0 0.0 0.0
- joint FR_X_joint: origin xyz=0.240292 -0.056 0 rpy=0 0 0 -> xyz=0.216 -0.048 0 rpy=0 0 0
- joint HL_FOOT_joint: origin xyz=0.0 0.0 -0.228 rpy=0.0 0.0 0.0 -> xyz=0.0 0.0 -0.24944 rpy=0.0 0.0 0.0
- joint HL_X_joint: origin xyz=-0.240292 0.056 0 rpy=0 0 0 -> xyz=-0.216 0.048 0 rpy=0 0 0
- joint HR_FOOT_joint: origin xyz=0.0 0.0 -0.228 rpy=0.0 0.0 0.0 -> xyz=0.0 0.0 -0.24944 rpy=0.0 0.0 0.0
- joint HR_X_joint: origin xyz=-0.240292 -0.056 0 rpy=0 0 0 -> xyz=-0.216 -0.048 0 rpy=0 0 0

Commit message: ✨ feat: urdf修正

File: config/robot.urdf (robot description, URDF)
Before this commit: robot bupt_dog, 17 links, 16 joints
Links:
- link FL_X: mass 1.440087 -> 1.5435
- link FR_X: mass 1.440087 -> 1.5435
- link HL_X: mass 1.440087 -> 1.5435
- link HR_X: mass 1.440087 -> 1.5435

Commit message: ✨ feat: urdf update

File: config/robot.urdf (robot description, URDF)
Before this commit: robot bupt_dog, 17 links, 16 joints
Links:
- link FL_FOOT: mass 0.06 -> 0.025
- link FL_X: mass 1.5435 -> 1.642
- link FR_FOOT: mass 0.06 -> 0.025
- link FR_X: mass 1.5435 -> 1.642
- link HL_FOOT: mass 0.06 -> 0.025
- link HL_X: mass 1.5435 -> 1.642
- link HR_FOOT: mass 0.06 -> 0.025
- link HR_X: mass 1.5435 -> 1.642

Commit message: ✨ feat: MPC效果良好

File: config/robot.urdf (robot description, URDF)
Before this commit: robot bupt_dog, 17 links, 16 joints
Links:
- added link base_link
- link FL_FOOT: mass 0.025 -> 0.009
- link FL_KNEE: mass 0.22 -> 0.14294956; geometry collision box size=0.02977 0.0225 0.18; visual box size=0.02977 0.0225 0.18
- link FL_Y: mass 0.272466 -> 0.24385482; geometry collision box size=0.044 0.033 0.18; visual box size=0.044 0.033 0.18
- link FR_FOOT: mass 0.025 -> 0.009
- link FR_KNEE: mass 0.22 -> 0.14294956; geometry collision box size=0.02977 0.0225 0.18; visual box size=0.02977 0.0225 0.18
- link FR_Y: mass 0.272466 -> 0.24385482; geometry collision box size=0.044 0.033 0.18; visual box size=0.044 0.033 0.18
- link HL_FOOT: mass 0.025 -> 0.009
- link HL_KNEE: mass 0.22 -> 0.14294956; geometry collision box size=0.02977 0.0225 0.18; visual box size=0.02977 0.0225 0.18
- link HL_Y: mass 0.272466 -> 0.24385482; geometry collision box size=0.044 0.033 0.18; visual box size=0.044 0.033 0.18
- link HR_FOOT: mass 0.025 -> 0.009
- link HR_KNEE: mass 0.22 -> 0.14294956; geometry collision box size=0.02977 0.0225 0.18; visual box size=0.02977 0.0225 0.18
- link HR_Y: mass 0.272466 -> 0.24385482; geometry collision box size=0.044 0.033 0.18; visual box size=0.044 0.033 0.18
Joints:
- added joint base: type fixed, parent base_link, child body
- joint FL_FOOT_joint: origin xyz=0.0 0.0 -0.24944 rpy=0.0 0.0 0.0 -> xyz=0.0 0.0 -0.18 rpy=0.0 0.0 0.0
- joint FL_KNEE_joint: origin xyz=0.0 0.0 -0.215 rpy=0.0 0.0 0.0 -> xyz=0.0 0.0 -0.18 rpy=0.0 0.0 0.0
- joint FL_Y_joint: origin xyz=0.0 0.1216 0.0 rpy=0.0 0.0 0.0 -> xyz=0.0 0.1171 0.0 rpy=0.0 0.0 0.0
- joint FR_FOOT_joint: origin xyz=0.0 0.0 -0.24944 rpy=0.0 0.0 0.0 -> xyz=0.0 0.0 -0.18 rpy=0.0 0.0 0.0
- joint FR_KNEE_joint: origin xyz=0.0 0.0 -0.215 rpy=0.0 0.0 0.0 -> xyz=0.0 0.0 -0.18 rpy=0.0 0.0 0.0
- joint FR_Y_joint: origin xyz=0.0 -0.1216 0.0 rpy=0.0 0.0 0.0 -> xyz=0.0 -0.1171 0.0 rpy=0.0 0.0 0.0
- joint HL_FOOT_joint: origin xyz=0.0 0.0 -0.24944 rpy=0.0 0.0 0.0 -> xyz=0.0 0.0 -0.18 rpy=0.0 0.0 0.0
- joint HL_KNEE_joint: origin xyz=0.0 0.0 -0.215 rpy=0.0 0.0 0.0 -> xyz=0.0 0.0 -0.18 rpy=0.0 0.0 0.0
- joint HL_Y_joint: origin xyz=0.0 0.1216 0.0 rpy=0.0 0.0 0.0 -> xyz=0.0 0.1171 0.0 rpy=0.0 0.0 0.0
- joint HR_FOOT_joint: origin xyz=0.0 0.0 -0.24944 rpy=0.0 0.0 0.0 -> xyz=0.0 0.0 -0.18 rpy=0.0 0.0 0.0
- joint HR_KNEE_joint: origin xyz=0.0 0.0 -0.215 rpy=0.0 0.0 0.0 -> xyz=0.0 0.0 -0.18 rpy=0.0 0.0 0.0
- joint HR_Y_joint: origin xyz=0.0 -0.1216 0.0 rpy=0.0 0.0 0.0 -> xyz=0.0 -0.1171 0.0 rpy=0.0 0.0 0.0

Commit message: 🎈 perf: 新机械结构调参

File: config/robot.urdf (robot description, URDF)
Before this commit: robot bupt_dog, 18 links, 17 joints
Links:
- link FL_X: mass 1.642 -> 1.464; geometry collision cylinder length=0.08861 radius=0.046; visual cylinder length=0.08861 radius=0.046
- link FR_X: mass 1.642 -> 1.464; geometry collision cylinder length=0.08861 radius=0.046; visual cylinder length=0.08861 radius=0.046
- link HL_X: mass 1.642 -> 1.464; geometry collision cylinder length=0.08861 radius=0.046; visual cylinder length=0.08861 radius=0.046
- link HR_X: mass 1.642 -> 1.464; geometry collision cylinder length=0.08861 radius=0.046; visual cylinder length=0.08861 radius=0.046
Joints:
- joint FL_X_joint: origin xyz=0.216 0.048 0 rpy=0 0 0 -> xyz=0.222 0.048 0 rpy=0 0 0
- joint FL_Y_joint: origin xyz=0.0 0.1171 0.0 rpy=0.0 0.0 0.0 -> xyz=0.0 0.08861 0.0 rpy=0.0 0.0 0.0
- joint FR_X_joint: origin xyz=0.216 -0.048 0 rpy=0 0 0 -> xyz=0.222 -0.048 0 rpy=0 0 0
- joint FR_Y_joint: origin xyz=0.0 -0.1171 0.0 rpy=0.0 0.0 0.0 -> xyz=0.0 -0.08861 0.0 rpy=0.0 0.0 0.0
- joint HL_X_joint: origin xyz=-0.216 0.048 0 rpy=0 0 0 -> xyz=-0.222 0.048 0 rpy=0 0 0
- joint HL_Y_joint: origin xyz=0.0 0.1171 0.0 rpy=0.0 0.0 0.0 -> xyz=0.0 0.08861 0.0 rpy=0.0 0.0 0.0
- joint HR_X_joint: origin xyz=-0.216 -0.048 0 rpy=0 0 0 -> xyz=-0.222 -0.048 0 rpy=0 0 0
- joint HR_Y_joint: origin xyz=0.0 -0.1171 0.0 rpy=0.0 0.0 0.0 -> xyz=0.0 -0.08861 0.0 rpy=0.0 0.0 0.0
